File: board/BoardyMcBoardFace.kicad_pcb (KiCad board)
At the start: 4 copper layers, 95 x 24 mm, 111 parts, among them J1 SMA, J2 ARM 10pin, J3 USB_B_Micro, J4 Conn_01x02_Male, J5 Conn_01x02_Male, SW1 SW_Push, U1 nRF24L01P, U2 STM32F103CBT6, U3 USBLC6-2SC6, U4 LM393, U5 AMS1117-5.0, U6 AMS1117-3.3, U7 USBLC6-2SC6, U8 USBLC6-2SC6, U9 TJA1051T-3, Y1 16MHz, Y2 16MHz

Commit message: move stuff aroud
Parts:
- removed C28, C31: 100n, Capacitor_SMD:C_0402_1005Metric
- removed D21, D22: WS2812B, LED_SMD:LED_WS2812B-2020_PLCC4_2.0x2.0mm
- added J6: Conn_01x02_Male, Connector_PinHeader_1.27mm:PinHeader_1x02_P1.27mm_Vertical, F.Cu at (187.6, 100.3)
- moved C3 13.7 mm to (172.0, 111.4)
- moved JP1 13.7 mm to (184.2, 100.2), turned to 0 degrees
- moved R3 12.5 mm to (182.1, 100.6)
- moved C2 9.60 mm to (181.4, 113.7), turned to -90 degrees
- moved C12 7.91 mm to (125.5, 104.4), turned to 180 degrees
- moved SW1 5.16 mm to (169.5, 111.2), turned to -90 degrees
- moved TP1 4.90 mm to (195.1, 108.4)
- moved C11 4.79 mm to (121.1, 110.0), turned to 90 degrees
- moved TP4 3.76 mm to (195.1, 113.0)
- moved JP2 3.10 mm to (165.9, 111.7), turned to 180 degrees
- moved C1 2.03 mm to (184.0, 104.8)
- moved C46 1.46 mm to (128.2, 111.3), turned to -90 degrees
- moved C20 1.45 mm to (186.5, 105.5), turned to 0 degrees
- moved C13 1.28 mm to (168.7, 114.5), turned to 180 degrees
- moved TP3 0.66 mm to (195.1, 110.7)
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Connections:
- D23 pad 2: Net-(D22-Pad4) -> /PIXEL_OFFBOARD
- U$1 pad P$29: /PIXEL_OFFBOARD -> unconnected-(U$1-PadP$29)
- U$1 pad P$31: /PIXEL_OFFBOARD -> unconnected-(U$1-PadP$31)
- U$1 pad P$45: unconnected-(U$1-PadP$45) -> /PIXEL_OFFBOARD
- U$1 pad P$47: unconnected-(U$1-PadP$47) -> /PIXEL_OFFBOARD
Routing:
- net Net-(D22-Pad4): track 28.0 -> 0.00 mm, vias 2 -> 0
- net /PIXEL_OFFBOARD: track 19.9 -> 41.5 mm, vias 0 -> 2
- net /CAN_H: track 11.7 -> 26.6 mm
- net +3V3: track 109.9 -> 99.3 mm, vias 47 -> 38
- net /CAN_L: track 11.0 -> 21.0 mm
- net GND: track 211.1 -> 203.1 mm, vias 102 -> 99
- net /NRST: track 32.6 -> 26.7 mm
- net /CAN_TX: track 21.4 -> 19.5 mm
- net Net-(D21-Pad4): track 1.88 -> 0.00 mm
- net /BOOT: track 15.5 -> 17.2 mm
- net Net-(JP1-Pad2): track 1.71 -> 2.90 mm
- net /PIXEL_MOSI: track 29.6 -> 28.5 mm
- net /RADIO_SPI_SCK: track 56.8 -> 55.9 mm
- net /RADIO_SPI_NSS: track 55.5 -> 54.8 mm
- net /CAN_RX: track 16.7 -> 16.1 mm
Other:
- board text added: "BALL DETECTOR"
- board text added: "RST"
- board text removed: "BALL"
- board text removed: "DETECTOR"
- board text removed: "TERM"
- board text removed: "VCC"

Commit message: final touches
Parts:
- removed TP1, TP3, TP4: TestPoint_Flag, TestPoint:TestPoint_Pad_1.0x1.0mm
- added C24: 100n, Capacitor_SMD:C_0402_1005Metric, F.Cu at (195.7, 109.3)
- added C28: 100n, Capacitor_SMD:C_0402_1005Metric, F.Cu at (192.4, 109.3)
- added D20: WS2812B, LED_SMD:LED_WS2812B-2020_PLCC4_2.0x2.0mm, F.Cu at (192.9, 111.1)
- added D21: WS2812B, LED_SMD:LED_WS2812B-2020_PLCC4_2.0x2.0mm, F.Cu at (196.2, 111.1)
- added D22: LED, LED_SMD:LED_0402_1005Metric, F.Cu at (183.0, 114.2)
- added D27: LED, LED_SMD:LED_0402_1005Metric, F.Cu at (193.9, 114.2)
- added D28: LED, LED_SMD:LED_0402_1005Metric, F.Cu at (175.9, 121.5)
- added R12: 1k, Resistor_SMD:R_0402_1005Metric, F.Cu at (192.9, 114.2)
- added R14: 1k, Resistor_SMD:R_0402_1005Metric, F.Cu at (174.9, 121.5)
- added R7: 1k, Resistor_SMD:R_0402_1005Metric, F.Cu at (184.0, 114.2)
- moved J2 12.0 mm to (187.6, 100.3), turned to -90 degrees
- moved JP1 11.3 mm to (193.7, 106.4), turned to -90 degrees
- moved J6 10.5 mm to (196.1, 106.4), turned to 90 degrees
- moved R3 10.2 mm to (190.7, 106.2)
- moved D5 0.48 mm to (190.4, 114.1)
- moved U7 0.43 mm to (185.6, 107.7)
- moved U3 0.38 mm to (185.6, 111.2)
- moved D6 0.38 mm to (186.6, 114.2)
- moved C20 0.23 mm to (186.3, 105.4)
Connections:
- D23 pad 2: /PIXEL_OFFBOARD -> Net-(D23-Pad2)
- U$1 pad P$21: /DRBL_PWM_1 -> /I2C1_SDA
- U$1 pad P$23: /DRBL_PWM_1 -> /I2C1_SDA
- U$1 pad P$25: /DRBL_PWM_2 -> /I2C1_SCL
- U$1 pad P$27: /DRBL_PWM_2 -> /I2C1_SCL
- U$1 pad P$31: unconnected-(U$1-PadP$31) -> /DRBL_PWM_1
- U$1 pad P$33: unconnected-(U$1-PadP$33) -> /DRBL_PWM_1
- U$1 pad P$35: /I2C1_SDA -> /DRBL_PWM_2
- U$1 pad P$37: /I2C1_SDA -> /DRBL_PWM_2
- U$1 pad P$39: /I2C1_SCL -> unconnected-(U$1-PadP$39)
- U$1 pad P$41: /I2C1_SCL -> /PIXEL_OFFBOARD
- U$1 pad P$43: unconnected-(U$1-PadP$43) -> /PIXEL_OFFBOARD
- U$1 pad P$45: /PIXEL_OFFBOARD -> unconnected-(U$1-PadP$45)
- U$1 pad P$47: /PIXEL_OFFBOARD -> unconnected-(U$1-PadP$47)
Routing:
- net Net-(D23-Pad2): track 0.00 -> 44.0 mm, vias 0 -> 2
- net /PIXEL_OFFBOARD: track 41.5 -> 11.1 mm, vias 2 -> 0
- net /SWDIO_CONN: track 3.62 -> 14.0 mm, vias 0 -> 1
- net /SWCLK_CONN: track 3.51 -> 12.0 mm, vias 0 -> 1
- net /CAN_H: track 26.6 -> 18.2 mm
- net GND: track 203.1 -> 211.3 mm, vias 99 -> 103
- net /TRACESWO_CONN: track 3.76 -> 10.9 mm, vias 0 -> 1
- net /NRST_CONN: track 3.86 -> 10.5 mm, vias 0 -> 1
- net +3V3: track 99.3 -> 105.2 mm
- net /CAN_L: track 21.0 -> 15.6 mm
- net /DRBL_PWM_2: track 30.9 -> 33.5 mm
- net /DRBL_PWM_1: track 31.0 -> 33.6 mm
- net /CAN_RX: track 16.1 -> 13.5 mm
- net /I2C1_SDA: track 27.5 -> 25.1 mm
- net /NRST: track 26.7 -> 24.5 mm
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Other:
- board text added: "The Bots Mainboard - Designed by Akhil V"
- board text removed: "3V"
- board text removed: "5V"

Commit message: finalized
Parts:
- FB1: footprint Inductor_SMD:L_0402_1005Metric -> Inductor_SMD:L_0805_2012Metric
- SW1: footprint Button_Switch_SMD:SW_Push_SPST_NO_Alps_SKRK -> ExtraStuff:TS-1187A-B-A-B
- moved JP2 4.33 mm to (163.1, 108.5), turned to 0 degrees
- moved C13 2.42 mm to (168.1, 116.8), turned to 0 degrees
- moved SW1 1.72 mm to (168.1, 112.3)
- moved C8 0.82 mm to (169.9, 104.0)
- moved FB1 0.81 mm to (171.3, 104.7)
- moved C24 0.13 mm to (195.7, 109.5)
- moved C28 0.13 mm to (192.4, 109.5)
- moved D20 0.13 mm to (192.9, 111.3)
- moved D21 0.13 mm to (196.2, 111.3)
Connections:
- JP2 pad 1: GND -> +3V3
- JP2 pad 3: +3V3 -> GND
Routing:
- net /NRST: track 24.5 -> 32.5 mm
- net GND: track 211.3 -> 218.5 mm, vias 103 -> 106
- net +3V3: track 105.2 -> 109.5 mm, vias 38 -> 39
- net /PIXEL_MOSI: track 28.5 -> 32.2 mm
- net /BOOT: track 17.7 -> 20.5 mm
