File: board/BoardyMcBoardFace.kicad_sch (KiCad schematic)
At the start: 111 parts, among them J1 SMA, J2 ARM 10pin, J3 USB_B_Micro, J4 Conn_01x02_Male, J5 Conn_01x02_Male, SW1 SW_Push, U1 nRF24L01P, U2 STM32F103CBT6, U3 USBLC6-2SC6, U4 LM393, U5 AMS1117-5.0, U6 AMS1117-3.3, U7 USBLC6-2SC6, U8 USBLC6-2SC6, U9 TJA1051T-3, Y1 16MHz, Y2 16MHz

Commit message: move stuff aroud
Parts:
- removed C28, C31: 100n, Capacitor_SMD:C_0402_1005Metric, symbol Device:C
- removed D21, D22: WS2812B, LED_SMD:LED_WS2812B-2020_PLCC4_2.0x2.0mm, symbol LED:WS2812B
- added J6: Conn_01x02_Male, Connector_PinHeader_1.27mm:PinHeader_1x02_P1.27mm_Vertical, symbol Connector:Conn_01x02_Male
Connections:
- net CAN_H: now also J6.1 (Pin_1)
- net CAN_L: now also J6.2 (Pin_2)
- net PIXEL_OFFBOARD: now also D23.2 (DOUT), U$1.P$45 (45), U$1.P$47 (47); no longer U$1.P$29 (29), U$1.P$31 (31)
Other:
- moved on the sheet: C32, C33, C34, C35, C36, C37, C38, C39, C40, C41, C42, C43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

Commit message: final touches
Parts:
- removed TP1, TP3, TP4: TestPoint_Flag, TestPoint:TestPoint_Pad_1.0x1.0mm, symbol Connector:TestPoint_Flag
- added C? (x2): 100n, Capacitor_SMD:C_0402_1005Metric, symbol Device:C
- added D20, D21: WS2812B, LED_SMD:LED_WS2812B-2020_PLCC4_2.0x2.0mm, symbol LED:WS2812B
- added D22, D27, D28: LED, LED_SMD:LED_0402_1005Metric, symbol Device:LED
- added R12, R14, R7: 1k, Resistor_SMD:R_0402_1005Metric, symbol Device:R
Connections:
- net +3V3: now also C?.1, C?.1, D20.1 (VDD), D21.1 (VDD), R7.1
- net +5V: now also R12.1
- net DRBL_PWM_1: now also U$1.P$31 (31), U$1.P$33 (33); no longer U$1.P$21 (21), U$1.P$23 (23)
- net DRBL_PWM_2: now also U$1.P$35 (35), U$1.P$37 (37); no longer U$1.P$25 (25), U$1.P$27 (27)
- net GND: now also C?.2, C?.2, D20.3 (VSS), D21.3 (VSS), D22.2 (A), D27.2 (A), D28.2 (A)
- net I2C1_SCL: now also U$1.P$25 (25), U$1.P$27 (27); no longer U$1.P$39 (39), U$1.P$41 (41)
- net I2C1_SDA: now also U$1.P$21 (21), U$1.P$23 (23); no longer U$1.P$35 (35), U$1.P$37 (37)
- net PIXEL_OFFBOARD: now also U$1.P$41 (41), U$1.P$43 (43), D20.2 (DOUT); no longer D23.2 (DOUT), U$1.P$45 (45), U$1.P$47 (47)
- net VBUS: now also R14.1
- new net: D22.1 (K), R7.2
- new net: D27.1 (K), R12.2
- new net: D20.4 (DIN), D21.2 (DOUT)
- new net: D21.4 (DIN), D23.2 (DOUT)
- new net: D28.1 (K), R14.2
Other:
- note added: "Power Leds"
- note removed: "Test Points"
- moved on the sheet: C32, C33, C34, C35, C36, C37, C38, C39, C40, C41, C42, C43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

Commit message: finalized
Parts:
- FB1: footprint Inductor_SMD:L_0402_1005Metric -> Inductor_SMD:L_0805_2012Metric
- SW1: footprint Button_Switch_SMD:SW_Push_SPST_NO_Alps_SKRK -> ExtraStuff:TS-1187A-B-A-B
- gave numbers to parts that had none: 2
Connections:
- net +3V3: now also JP2.1 (A); no longer JP2.3 (B)
- net GND: now also JP2.3 (B); no longer JP2.1 (A)
Changed lines of the file:
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@@
     (stroke (width 0) (type default) (color 0 0 0 0))
   )
-  (wire (pts (xy 247.015 138.43) (xy 254 138.43))
-    (stroke (width 0) (type default) (color 0 0 0 0))
-  )
   (wire (pts (xy 337.82 25.4) (xy 337.82 24.765))
     (stroke (width 0) (type default) (color 0 0 0 0))
@@
     (stroke (width 0) (type default) (color 0 0 0 0))
   )
-  (wire (pts (xy 226.695 138.43) (xy 234.315 138.43))
-    (stroke (width 0) (type default) (color 0 0 0 0))
-  )
   (wire (pts (xy 377.19 177.165) (xy 377.19 161.925))
     (stroke (width 0) (type default) (color 0 0 0 0))
@@
     (effects (font (size 1.27 1.27)) (justify right bottom))
   )
-  (label "BOOT" (at 240.665 142.24 270)
+  (label "BOOT" (at 235.077 142.875 270)
     (effects (font (size 1.2446 1.2446)) (justify right bottom))
   )
@@
     (property "Reference" "FB1" (id 0) (at 199.39 27.305 90))
     (property "Value" "120R" (id 1) (at 199.39 16.3068 90))
-    (property "Footprint" "Inductor_SMD:L_0402_1005Metric" (id 2) (at 199.39 19.177 90)
+    (property "Footprint" "Inductor_SMD:L_0805_2012Metric" (id 2) (at 199.39 19.177 90)
       (effects (font (size 1.27 1.27)) hide)
     )
@@
     (pin "1")
   )
-  (symbol (lib_id "power:GND") (at 226.695 138.43 180) (unit 1)
+  (symbol (lib_id "power:GND") (at 241.427 139.065 0) (unit 1)
     (in_bom yes) (on_board yes)
-    (property "Reference" "#PWR034" (id 0) (at 226.695 132.08 0)
+    (property "Reference" "#PWR034" (id 0) (at 241.427 145.415 0)
       (effects (font (size 1.27 1.27)) hide)
     )
-    (property "Value" "GND" (id 1) (at 226.568 134.0358 0))
-    (property "Footprint" "" (id 2) (at 226.695 138.43 0)
+    (property "Value" "GND" (id 1) (at 241.554 143.4592 0))
+    (property "Footprint" "" (id 2) (at 241.427 139.065 0)
       (effects (font (size 1.27 1.27)) hide)
     )
-    (property "Datasheet" "" (id 3) (at 226.695 138.43 0)
+    (property "Datasheet" "" (id 3) (at 241.427 139.065 0)
       (effects (font (size 1.27 1.27)) hide)
     )
@@
       (effects (font (size 1.27 1.27)) (justify right))
     )
-    (property "Footprint" "Button_Switch_SMD:SW_Push_SPST_NO_Alps_SKRK" (id 2) (at 25.4 36.83 0)
+    (property "Footprint" "ExtraStuff:TS-1187A-B-A-B" (id 2) (at 25.4 36.83 0)
       (effects (font (size 1.27 1.27)) hide)
     )
@@
     (pin "2")
   )
-  (symbol (lib_id "power:+3.3V") (at 254 138.43 0) (unit 1)
+  (symbol (lib_id "power:+3.3V") (at 228.727 139.065 0) (unit 1)
     (in_bom yes) (on_board yes)
-    (property "Reference" "#PWR035" (id 0) (at 254 142.24 0)
+    (property "Reference" "#PWR035" (id 0) (at 228.727 142.875 0)
       (effects (font (size 1.27 1.27)) hide)
     )
-    (property "Value" "+3.3V" (id 1) (at 254.635 133.985 0))
-    (property "Footprint" "" (id 2) (at 254 138.43 0)
+    (property "Value" "+3.3V" (id 1) (at 229.362 134.62 0))
+    (property "Footprint" "" (id 2) (at 228.727 139.065 0)
       (effects (font (size 1.27 1.27)) hide)
     )
-    (property "Datasheet" "" (id 3) (at 254 138.43 0)
+    (property "Datasheet" "" (id 3) (at 228.727 139.065 0)
       (effects (font (size 1.27 1.27)) hide)
     )
@@
     (pin "1")
   )
+  (symbol (lib_id "Jumper:Jumper_3_Open") (at 235.077 139.065 0) (unit 1)
+    (in_bom yes) (on_board yes)
+    (property "Reference" "JP2" (id 0) (at 240.03 132.461 0))
+    (property "Value" "Jumper_3_Open" (id 1) (at 245.491 134.366 0))
+    (property "Footprint" "Connector_PinHeader_1.27mm:PinHeader_1x03_P1.27mm_Vertical" (id 2) (at 235.077 139.065 0)
+      (effects (font (size 1.27 1.27)) hide)
+    )
+    (property "Datasheet" "~" (id 3) (at 235.077 139.065 0)
+      (effects (font (size 1.27 1.27)) hide)
+    )
+    (pin "1")
+    (pin "2")
+    (pin "3")
+  )
   (symbol (lib_id "power:GND") (at 231.14 26.797 0) (unit 1)
     (in_bom yes) (on_board yes)
@@
   (symbol (lib_id "Device:C") (at 289.687 196.723 0) (unit 1)
     (in_bom yes) (on_board yes)
-    (property "Reference" "C?" (id 0) (at 287.528 191.897 0)
+    (property "Reference" "C28" (id 0) (at 287.528 191.897 0)
       (effects (font (size 1.27 1.27)) (justify left))
     )
@@
   (symbol (lib_id "Device:C") (at 284.226 196.723 0) (unit 1)
     (in_bom yes) (on_board yes)
-    (property "Reference" "C?" (id 0) (at 282.956 191.77 0)
+    (property "Reference" "C24" (id 0) (at 282.956 191.77 0)
       (effects (font (size 1.27 1.27)) (justify left))
     )
@@
     (pin "1")
   )
-  (symbol (lib_id "Jumper:Jumper_3_Open") (at 240.665 138.43 0) (unit 1)
-    (in_bom yes) (on_board yes) (fields_autoplaced)
-    (property "Reference" "JP2" (id 0) (at 240.665 132.08 0))
-    (property "Value" "Jumper_3_Open" (id 1) (at 240.665 134.62 0))
-    (property "Footprint" "Connector_PinHeader_1.27mm:PinHeader_1x03_P1.27mm_Vertical" (id 2) (at 240.665 138.43 0)
-      (effects (font (size 1.27 1.27)) hide)
-    )
-    (property "Datasheet" "~" (id 3) (at 240.665 138.43 0)
-      (effects (font (size 1.27 1.27)) hide)
-    )
-    (pin "1")
-    (pin "2")
-    (pin "3")
-  )
   (sheet_instances
     (path "/" (page "1"))
@@
       (reference "C23") (unit 1) (value "4p7") (footprint "Capacitor_SMD:C_0402_1005Metric")
     )
+    (path "/d137c7a3-2f97-4a30-97e4-3ac71acf22c5"
+      (reference "C24") (unit 1) (value "100n") (footprint "Capacitor_SMD:C_0402_1005Metric")
+    )
     (path "/00000000-0000-0000-0000-0000645faf38"
       (reference "C25") (unit 1) (value "10n") (footprint "Capacitor_SMD:C_0402_1005Metric")
@@
       (reference "C27") (unit 1) (value "22u") (footprint "Capacitor_SMD:C_0805_2012Metric")
     )
+    (path "/c09e5454-6031-4bf3-a6ec-f677e6630c9d"
+      (reference "C28") (unit 1) (value "100n") (footprint "Capacitor_SMD:C_0402_1005Metric")
+    )
     (path "/00000000-0000-0000-0000-0000647dc1e4"
       (reference "C29") (unit 1) (value "10n") (footprint "Capacitor_SMD:C_0402_1005Metric")
@@
       (reference "C46") (unit 1) (value "100n") (footprint "Capacitor_SMD:C_0402_1005Metric")
     )
-    (path "/c09e5454-6031-4bf3-a6ec-f677e6630c9d"
-      (reference "C?") (unit 1) (value "100n") (footprint "Capacitor_SMD:C_0402_1005Metric")
-    )
-    (path "/d137c7a3-2f97-4a30-97e4-3ac71acf22c5"
-      (reference "C?") (unit 1) (value "100n") (footprint "Capacitor_SMD:C_0402_1005Metric")
-    )
     (path "/5e19ece2-1c3b-4824-944b-dfe6e8d09f84"
       (reference "D1") (unit 1) (value "WS2812B") (footprint "LED_SMD:LED_WS2812B-2020_PLCC4_2.0x2.0mm")
@@
     )
     (path "/00000000-0000-0000-0000-0000633ce523"
-      (reference "FB1") (unit 1) (value "120R") (footprint "Inductor_SMD:L_0402_1005Metric")
+      (reference "FB1") (unit 1) (value "120R") (footprint "Inductor_SMD:L_0805_2012Metric")
     )
     (path "/aaf5514b-b038-4843-922e-cdb434b65db4"
@@
       (reference "JP1") (unit 1) (value "Jumper_2_Open") (footprint "Connector_PinHeader_1.27mm:PinHeader_1x02_P1.27mm_Vertical")
     )
-    (path "/ff7396d4-7561-4910-9c0d-d4d11560877f"
+    (path "/2d523b82-e342-4b3f-8985-0307c7a62995"
       (reference "JP2") (unit 1) (value "Jumper_3_Open") (footprint "Connector_PinHeader_1.27mm:PinHeader_1x03_P1.27mm_Vertical")
     )
@@
     )
     (path "/00000000-0000-0000-0000-000066245539"
-      (reference "SW1") (unit 1) (value "SW_Push") (footprint "Button_Switch_SMD:SW_Push_SPST_NO_Alps_SKRK")
+      (reference "SW1") (unit 1) (value "SW_Push") (footprint "ExtraStuff:TS-1187A-B-A-B")
     )
     (path "/56fb8db9-d85c-45ae-a2c2-f865f8ec3859"
